Commit message: Updated descriptions to use sub namespace

File: robots/sub_default.xacro (robot description, xacro)
@@ -17,13 +17,13 @@
      limitations under the License.
 -->
-<robot name="rexrov" xmlns:xacro="http://www.ros.org/wiki/xacro" >
+<robot name="sub" xmlns:xacro="http://www.ros.org/wiki/xacro" >
   <xacro:arg name="debug" default="0"/>
-  <xacro:arg name="namespace" default="rexrov"/>
+  <xacro:arg name="namespace" default="sub"/>
   <xacro:arg name="inertial_reference_frame" default="world"/>
   <!-- Include the ROV macro file -->
-  <xacro:include filename="$(find uuv_descriptions)/urdf/rexrov_base.xacro"/>
-  <xacro:include filename="$(find uuv_descriptions)/urdf/rexrov.gazebo.xacro"/>
-  <!-- Create the rexrov -->
-  <xacro:rexrov_base
+  <xacro:include filename="$(find sub_descriptions)/urdf/sub_base.xacro"/>
+  <xacro:include filename="$(find sub_descriptions)/urdf/sub.gazebo.xacro"/>
+  <!-- Create the sub -->
+  <xacro:sub_base
     namespace="$(arg namespace)"
     inertial_reference_frame="$(arg inertial_reference_frame)">
@@ -36,8 +36,8 @@
         <debug>$(arg debug)</debug>
         <!-- Adding the hydrodynamic and hydrostatic parameters for the vehicle-->
-        <xacro:rexrov_hydro_model namespace="$(arg namespace)"/>
+        <xacro:sub_hydro_model namespace="$(arg namespace)"/>
       </plugin>
     </gazebo>
-  </xacro:rexrov_base>
+  </xacro:sub_base>
   <!-- Joint state publisher plugin -->
   <xacro:default_joint_state_publisher namespace="$(arg namespace)" update_rate="50"/>

File: robots/sub_default_noisy_pose.xacro (robot description, xacro)
@@ -17,13 +17,15 @@
      limitations under the License.
 -->
-<robot name="rexrov" xmlns:xacro="http://www.ros.org/wiki/xacro" >
+<robot name="sub" xmlns:xacro="http://www.ros.org/wiki/xacro" >
   <xacro:arg name="debug" default="0"/>
-  <xacro:arg name="namespace" default="rexrov"/>
+  <xacro:arg name="namespace" default="sub"/>
+  <xacro:arg name="noise_amp" default="0.02"/>
+  <xacro:arg name="noise_sigma" default="0.002"/>
   <xacro:arg name="inertial_reference_frame" default="world"/>
   <!-- Include the ROV macro file -->
-  <xacro:include filename="$(find uuv_descriptions)/urdf/rexrov_base.xacro"/>
-  <xacro:include filename="$(find uuv_descriptions)/urdf/rexrov.gazebo.xacro"/>
-  <!-- Create the rexrov -->
-  <xacro:rexrov_base
+  <xacro:include filename="$(find uuv_descriptions)/urdf/sub_base.xacro"/>
+  <xacro:include filename="$(find uuv_descriptions)/urdf/sub.gazebo.xacro"/>
+  <!-- Create the sub -->
+  <xacro:sub_base
     namespace="$(arg namespace)"
     inertial_reference_frame="$(arg inertial_reference_frame)">
@@ -36,17 +38,16 @@
         <debug>$(arg debug)</debug>
         <!-- Adding the hydrodynamic and hydrostatic parameters for the vehicle-->
-        <xacro:rexrov_hydro_model namespace="$(arg namespace)"/>
-      </plugin>
-      <plugin name="imu_plugin" filename="libgazebo_ros_imu.so">
-        <alwaysOn>true</alwaysOn>
-        <bodyName>base_footprint</bodyName>
-        <topicName>imu</topicName>
-        <serviceName>imu_service</serviceName>
-        <gaussianNoise>0.1</gaussianNoise>
-        <updateRate>20.0</updateRate>
+        <xacro:sub_hydro_model namespace="$(arg namespace)"/>
       </plugin>
     </gazebo>
-  </xacro:rexrov_base>
+  </xacro:sub_base>
   <!-- Joint state publisher plugin -->
   <xacro:default_joint_state_publisher namespace="$(arg namespace)" update_rate="50"/>
+  <!-- Add pose_gt with Gaussian noise -->
+  <xacro:pose_3d_sensor namespace="$(arg namespace)"
+                        suffix="noisy"
+                        parent_link="$(arg namespace)/base_link"
+                        gaussian_noise_amplitude="$(arg noise_amp)"
+                        gaussian_noise_sigma="$(arg noise_sigma)"
+                        topic="pose_gt_noisy" />
 </robot>

File: robots/sub_imu.xacro (robot description, xacro)
@@ -17,15 +17,13 @@
      limitations under the License.
 -->
-<robot name="rexrov" xmlns:xacro="http://www.ros.org/wiki/xacro" >
+<robot name="sub" xmlns:xacro="http://www.ros.org/wiki/xacro" >
   <xacro:arg name="debug" default="0"/>
-  <xacro:arg name="namespace" default="rexrov"/>
-  <xacro:arg name="noise_amp" default="0.02"/>
-  <xacro:arg name="noise_sigma" default="0.002"/>
+  <xacro:arg name="namespace" default="sub"/>
   <xacro:arg name="inertial_reference_frame" default="world"/>
   <!-- Include the ROV macro file -->
-  <xacro:include filename="$(find uuv_descriptions)/urdf/rexrov_base.xacro"/>
-  <xacro:include filename="$(find uuv_descriptions)/urdf/rexrov.gazebo.xacro"/>
-  <!-- Create the rexrov -->
-  <xacro:rexrov_base
+  <xacro:include filename="$(find sub_descriptions)/urdf/sub_base.xacro"/>
+  <xacro:include filename="$(find sub_descriptions)/urdf/sub.gazebo.xacro"/>
+  <!-- Create the sub -->
+  <xacro:sub_base
     namespace="$(arg namespace)"
     inertial_reference_frame="$(arg inertial_reference_frame)">
@@ -38,16 +36,17 @@
         <debug>$(arg debug)</debug>
         <!-- Adding the hydrodynamic and hydrostatic parameters for the vehicle-->
-        <xacro:rexrov_hydro_model namespace="$(arg namespace)"/>
+        <xacro:sub_hydro_model namespace="$(arg namespace)"/>
+      </plugin>
+      <plugin name="imu_plugin" filename="libgazebo_ros_imu.so">
+        <alwaysOn>true</alwaysOn>
+        <bodyName>base_footprint</bodyName>
+        <topicName>imu</topicName>
+        <serviceName>imu_service</serviceName>
+        <gaussianNoise>0.1</gaussianNoise>
+        <updateRate>20.0</updateRate>
       </plugin>
     </gazebo>
-  </xacro:rexrov_base>
+  </xacro:sub_base>
   <!-- Joint state publisher plugin -->
   <xacro:default_joint_state_publisher namespace="$(arg namespace)" update_rate="50"/>
-  <!-- Add pose_gt with Gaussian noise -->
-  <xacro:pose_3d_sensor namespace="$(arg namespace)"
-                        suffix="noisy"
-                        parent_link="$(arg namespace)/base_link"
-                        gaussian_noise_amplitude="$(arg noise_amp)"
-                        gaussian_noise_sigma="$(arg noise_sigma)"
-                        topic="pose_gt_noisy" />
 </robot>

File: urdf/sub.gazebo.xacro (robot description, xacro)
@@ -26,5 +26,5 @@
     <!-- Volume, see p.31 in Berg2012 -->
     <xacro:property name="volume" value="1.83826"/>
-    <xacro:macro name="rexrov_hydro_model" params="namespace">
+    <xacro:macro name="sub_hydro_model" params="namespace">
         <link name="${namespace}/base_link">
             <neutrally_buoyant>0</neutrally_buoyant>

File: urdf/sub_actuators.xacro (robot description, xacro)
@@ -18,5 +18,5 @@
 -->
 <robot xmlns:xacro="http://www.ros.org/wiki/xacro">
-  <xacro:property name="prop_mesh_file" value="file://$(find uuv_descriptions)/meshes/prop.dae"/>
+  <xacro:property name="prop_mesh_file" value="file://$(find sub_descriptions)/meshes/prop.dae"/>
   <!-- Thruster joint and link snippet -->
   <xacro:macro name="thruster_macro"

File: urdf/sub_base.xacro (robot description, xacro)
@@ -27,14 +27,14 @@
   -->
   <!-- includes -->
-  <xacro:include filename="$(find uuv_descriptions)/urdf/common.urdf.xacro"/>
+  <xacro:include filename="$(find sub_descriptions)/urdf/common.urdf.xacro"/>
   <xacro:include filename="$(find uuv_sensor_ros_plugins)/urdf/sensor_snippets.xacro"/>
   <xacro:include filename="$(find uuv_gazebo_ros_plugins)/urdf/snippets.xacro"/>
   <!-- Parameters -->
-  <xacro:property name="namespace" value="rexrov"/>
-  <xacro:property name="visual_mesh_file" value="file://$(find uuv_descriptions)/meshes/RexROV_no_props.dae"/>
-  <xacro:property name="prop_mesh_file" value="file://$(find uuv_descriptions)/meshes/prop.dae"/>
+  <xacro:property name="namespace" value="sub"/>
+  <xacro:property name="visual_mesh_file" value="file://$(find sub_descriptions)/meshes/RexROV_no_props.dae"/>
+  <xacro:property name="prop_mesh_file" value="file://$(find sub_descriptions)/meshes/prop.dae"/>
   <!-- Mass, see p.28 in Berg2012 -->
   <xacro:property name="mass" value="1862.87"/>
-  <xacro:macro name="rexrov_base" params="namespace *gazebo inertial_reference_frame">
+  <xacro:macro name="sub_base" params="namespace *gazebo inertial_reference_frame">
     <!-- base_link according to ROS conventions: x forward, z up -->
     <link name="${namespace}/base_link">
@@ -80,6 +80,6 @@
       </plugin>
     </gazebo> -->
-    <xacro:include filename="$(find uuv_descriptions)/urdf/rexrov_actuators.xacro"/>
-    <xacro:include filename="$(find uuv_descriptions)/urdf/rexrov_sensors.xacro"/>
+    <xacro:include filename="$(find sub_descriptions)/urdf/sub_actuators.xacro"/>
+    <xacro:include filename="$(find sub_descriptions)/urdf/sub_sensors.xacro"/>
   </xacro:macro>
 </robot>

File: urdf/sub_sensors.xacro (robot description, xacro)
@@ -52,6 +52,4 @@
     <origin xyz="1.15 0.63 0.4" rpy="0 0.6 -0.4"/>
   </xacro:default_camera>
-  <!-- Mount a GPS. -->
-  <xacro:default_gps namespace="${namespace}" parent_link="${namespace}/base_link" />
   <!-- Mount a Pose 3D sensor. -->
   <xacro:default_pose_3d_macro
